File: hardware/current_sink_dev.kicad_sch (KiCad schematic)
At the start: 0 parts

Commit message: Updates to structure of the schematic. Minor funcitonality adjustments.
Parts:
- added J2: ~, Connector_PinHeader_2.54mm:PinHeader_1x02_P2.54mm_Vertical, symbol Connector:Conn_01x02_Socket
Connections:
- new net GND: J2.2 (Pin_2)
- no-connect marks 3 -> 0
Other:
- removed sheet current_sink_stage1
- sheet current_setting ports: added none; removed curr_set_A_uC, curr_set_B_uC, set_curr_A, set_curr_B, supply_pos
- sheet current_sink_stage ports: added none; removed supply_neg, supply_pos, voltage_set_ss, voltage_sink
- sheet supply_gen ports: added none; removed supply_neg, supply_pos
Changed lines of the file:
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@@
 (kicad_sch (version 20230121) (generator eeschema)
   (paper "A3")
-  (junction (at 220.98 101.6) (diameter 0) (color 0 0 0 0)
-  )
-  (junction (at 205.74 101.6) (diameter 0) (color 0 0 0 0)
-  )
-  (junction (at 217.17 110.49) (diameter 0) (color 0 0 0 0)
-  )
-  (no_connect (at 217.17 118.11))
-  (no_connect (at 205.74 110.49))
-  (no_connect (at 220.98 118.11))
-  (wire (pts (xy 97.79 110.49) (xy 217.17 110.49))
+  (wire (pts (xy 218.44 104.14) (xy 218.44 110.49))
     (stroke (width 0) (type default))
   )
-  (wire (pts (xy 190.5 158.75) (xy 228.6 158.75))
+  (wire (pts (xy 223.52 104.14) (xy 218.44 104.14))
     (stroke (width 0) (type default))
   )
-  (wire (pts (xy 97.79 101.6) (xy 205.74 101.6))
-    (stroke (width 0) (type default))
+  (symbol (lib_id "power:GND") (at 218.44 110.49 0) (unit 1)
+    (in_bom yes) (on_board yes) (dnp no) (fields_autoplaced)
+    (property "Reference" "#PWR033" (at 218.44 116.84 0)
+      (effects (font (size 1.27 1.27)) hide)
+    )
+    (property "Value" "GND" (at 218.44 114.935 0)
+      (effects (font (size 1.27 1.27)))
+    )
+    (property "Footprint" "" (at 218.44 110.49 0)
+      (effects (font (size 1.27 1.27)) hide)
+    )
+    (property "Datasheet" "" (at 218.44 110.49 0)
+      (effects (font (size 1.27 1.27)) hide)
+    )
+    (pin "1")
+    (instances
+      (project "current_sink_dev"
+        (path "/695b42ec-77e0-4be3-bf4d-1fc5cfcb9ef1"
+          (reference "#PWR033") (unit 1)
+        )
+        (path "/695b42ec-77e0-4be3-bf4d-1fc5cfcb9ef1/02da786d-4b46-4498-8c46-331dfb2a8a58"
+          (reference "#PWR04") (unit 1)
+        )
+      )
+    )
   )
-  (wire (pts (xy 228.6 142.24) (xy 220.98 142.24))
-    (stroke (width 0) (type default))
-  )
-  (wire (pts (xy 190.5 139.7) (xy 205.74 139.7))
-    (stroke (width 0) (type default))
-  )
-  (wire (pts (xy 209.55 153.67) (xy 209.55 118.11))
-    (stroke (width 0) (type default))
-  )
-  (wire (pts (xy 205.74 139.7) (xy 205.74 101.6))
-    (stroke (width 0) (type default))
-  )
-  (wire (pts (xy 220.98 101.6) (xy 228.6 101.6))
-    (stroke (width 0) (type default))
-  )
-  (wire (pts (xy 217.17 110.49) (xy 217.17 151.13))
-    (stroke (width 0) (type default))
-  )
-  (wire (pts (xy 220.98 142.24) (xy 220.98 101.6))
-    (stroke (width 0) (type default))
-  )
-  (wire (pts (xy 209.55 118.11) (xy 228.6 118.11))
-    (stroke (width 0) (type default))
-  )
-  (wire (pts (xy 302.26 142.24) (xy 302.26 101.6))
-    (stroke (width 0) (type default))
-  )
-  (wire (pts (xy 289.56 142.24) (xy 302.26 142.24))
-    (stroke (width 0) (type default))
-  )
-  (wire (pts (xy 217.17 151.13) (xy 228.6 151.13))
-    (stroke (width 0) (type default))
-  )
-  (wire (pts (xy 190.5 153.67) (xy 209.55 153.67))
-    (stroke (width 0) (type default))
-  )
-  (wire (pts (xy 217.17 110.49) (xy 228.6 110.49))
-    (stroke (width 0) (type default))
-  )
-  (wire (pts (xy 205.74 101.6) (xy 220.98 101.6))
-    (stroke (width 0) (type default))
-  )
-  (wire (pts (xy 302.26 101.6) (xy 289.56 101.6))
-    (stroke (width 0) (type default))
+  (symbol (lib_id "Connector:Conn_01x02_Socket") (at 228.6 101.6 0) (unit 1)
+    (in_bom yes) (on_board yes) (dnp no) (fields_autoplaced)
+    (property "Reference" "J2" (at 229.87 103.505 0)
+      (effects (font (size 1.27 1.27)) (justify left))
+    )
+    (property "Value" "~" (at 229.87 104.775 0)
+      (effects (font (size 1.27 1.27)) (justify left))
+    )
+    (property "Footprint" "Connector_PinHeader_2.54mm:PinHeader_1x02_P2.54mm_Vertical" (at 228.6 101.6 0)
+      (effects (font (size 1.27 1.27)) hide)
+    )
+    (property "Datasheet" "~" (at 228.6 101.6 0)
+      (effects (font (size 1.27 1.27)) hide)
+    )
+    (pin "1")
+    (pin "2")
+    (instances
+      (project "current_sink_dev"
+        (path "/695b42ec-77e0-4be3-bf4d-1fc5cfcb9ef1"
+          (reference "J2") (unit 1)
+        )
+      )
+    )
   )
   (sheet (at 40.64 93.98) (size 57.15 29.21) (fields_autoplaced)
@@
       (effects (font (size 1.27 1.27)) (justify left top))
     )
-    (pin "supply_pos" bidirectional (at 97.79 101.6 0)
-      (effects (font (size 1.27 1.27)) (justify right))
-    )
-    (pin "supply_neg" bidirectional (at 97.79 110.49 0)
-      (effects (font (size 1.27 1.27)) (justify right))
-    )
     (instances
       (project "current_sink_dev"
@@
     )
   )
-  (sheet (at 228.6 93.98) (size 60.96 29.21) (fields_autoplaced)
+  (sheet (at 129.54 93.98) (size 60.96 29.21) (fields_autoplaced)
     (stroke (width 0.1524) (type solid))
     (fill (color 0 0 0 0.0000))
-    (property "Sheetname" "current_sink_stage" (at 228.6 93.2684 0)
+    (property "Sheetname" "current_sink_stage" (at 129.54 93.2684 0)
       (effects (font (size 1.27 1.27)) (justify left bottom))
     )
-    (property "Sheetfile" "current_sink_stage.kicad_sch" (at 228.6 123.7746 0)
+    (property "Sheetfile" "current_sink_stage.kicad_sch" (at 129.54 123.7746 0)
       (effects (font (size 1.27 1.27)) (justify left top))
-    )
-    (pin "voltage_sink" input (at 289.56 101.6 0)
-      (effects (font (size 1.27 1.27)) (justify right))
-    )
-    (pin "supply_neg" bidirectional (at 228.6 110.49 180)
-      (effects (font (size 1.27 1.27)) (justify left))
-    )
-    (pin "supply_pos" bidirectional (at 228.6 101.6 180)
-      (effects (font (size 1.27 1.27)) (justify left))
-    )
-    (pin "voltage_set_ss" output (at 228.6 118.11 180)
-      (effects (font (size 1.27 1.27)) (justify left))
     )
     (instances
@@
     )
   )
-  (sheet (at 228.6 134.62) (size 60.96 29.21) (fields_autoplaced)
+  (sheet (at 129.54 134.62) (size 60.96 29.21) (fields_autoplaced)
     (stroke (width 0.1524) (type solid))
     (fill (color 0 0 0 0.0000))
-    (property "Sheetname" "current_sink_stage1" (at 228.6 133.9084 0)
+    (property "Sheetname" "current_setting" (at 129.54 133.9084 0)
       (effects (font (size 1.27 1.27)) (justify left bottom))
     )
-    (property "Sheetfile" "current_sink_stage.kicad_sch" (at 228.6 164.4146 0)
+    (property "Sheetfile" "current_setting.kicad_sch" (at 129.54 164.4146 0)
       (effects (font (size 1.27 1.27)) (justify left top))
     )
-    (pin "voltage_sink" input (at 289.56 142.24 0)
-      (effects (font (size 1.27 1.27)) (justify right))
-    )
-    (pin "supply_neg" bidirectional (at 228.6 151.13 180)
-      (effects (font (size 1.27 1.27)) (justify left))
-    )
-    (pin "supply_pos" bidirectional (at 228.6 142.24 180)
-      (effects (font (size 1.27 1.27)) (justify left))
-    )
-    (pin "voltage_set_ss" output (at 228.6 158.75 180)
-      (effects (font (size 1.27 1.27)) (justify left))
-    )
     (instances
-      (project "current_sink_dev"
-        (path "/695b42ec-77e0-4be3-bf4d-1fc5cfcb9ef1" (page "3"))
-      )
-    )
-  )
-  (sheet (at 133.35 134.62) (size 57.15 29.21) (fields_autoplaced)
-    (stroke (width 0.1524) (type solid))
-    (fill (color 0 0 0 0.0000))
-    (property "Sheetname" "current_setting" (at 133.35 133.9084 0)
-      (effects (font (size 1.27 1.27)) (justify left bottom))
-    )
-    (property "Sheetfile" "current_setting.kicad_sch" (at 133.35 164.4146 0)
-      (effects (font (size 1.27 1.27)) (justify left top))
-    )
-    (pin "set_curr_A" output (at 190.5 153.67 0)
-      (effects (font (size 1.27 1.27)) (justify right))
-    )
-    (pin "curr_set_B_uC" output (at 133.35 158.75 180)
-      (effects (font (size 1.27 1.27)) (justify left))
-    )
-    (pin "set_curr_B" output (at 190.5 158.75 0)
-      (effects (font (size 1.27 1.27)) (justify right))
-    )
-    (pin "curr_set_A_uC" output (at 133.35 153.67 180)
-      (effects (font (size 1.27 1.27)) (justify left))
-    )
-    (pin "supply_pos" bidirectional (at 190.5 139.7 0)
-      (effects (font (size 1.27 1.27)) (justify right))
-    )
-    (instances

Commit message: Began initial routing. Schematic still not fully complete.
Parts:
- removed J2: ~, Connector_PinHeader_2.54mm:PinHeader_1x02_P2.54mm_Vertical, symbol Connector:Conn_01x02_Socket
Other:
- added sheet LCD_screen (LCD_screen.kicad_sch)
- added sheet mechanical_components (mechanical_components.kicad_sch)
Changed lines of the file:
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@@
 (kicad_sch (version 20230121) (generator eeschema)
   (paper "A3")
-  (wire (pts (xy 218.44 104.14) (xy 218.44 110.49))
-    (stroke (width 0) (type default))
-  )
-  (wire (pts (xy 223.52 104.14) (xy 218.44 104.14))
-    (stroke (width 0) (type default))
-  )
-  (symbol (lib_id "power:GND") (at 218.44 110.49 0) (unit 1)
-    (in_bom yes) (on_board yes) (dnp no) (fields_autoplaced)
-    (property "Reference" "#PWR033" (at 218.44 116.84 0)
-      (effects (font (size 1.27 1.27)) hide)
-    )
-    (property "Value" "GND" (at 218.44 114.935 0)
-      (effects (font (size 1.27 1.27)))
-    )
-    (property "Footprint" "" (at 218.44 110.49 0)
-      (effects (font (size 1.27 1.27)) hide)
-    )
-    (property "Datasheet" "" (at 218.44 110.49 0)
-      (effects (font (size 1.27 1.27)) hide)
-    )
-    (pin "1")
-    (instances
-      (project "current_sink_dev"
-        (path "/695b42ec-77e0-4be3-bf4d-1fc5cfcb9ef1"
-          (reference "#PWR033") (unit 1)
-        )
-        (path "/695b42ec-77e0-4be3-bf4d-1fc5cfcb9ef1/02da786d-4b46-4498-8c46-331dfb2a8a58"
-          (reference "#PWR04") (unit 1)
-        )
-      )
-    )
-  )
-  (symbol (lib_id "Connector:Conn_01x02_Socket") (at 228.6 101.6 0) (unit 1)
-    (in_bom yes) (on_board yes) (dnp no) (fields_autoplaced)
-    (property "Reference" "J2" (at 229.87 103.505 0)
-      (effects (font (size 1.27 1.27)) (justify left))
-    )
-    (property "Value" "~" (at 229.87 104.775 0)
-      (effects (font (size 1.27 1.27)) (justify left))
-    )
-    (property "Footprint" "Connector_PinHeader_2.54mm:PinHeader_1x02_P2.54mm_Vertical" (at 228.6 101.6 0)
-      (effects (font (size 1.27 1.27)) hide)
-    )
-    (property "Datasheet" "~" (at 228.6 101.6 0)
-      (effects (font (size 1.27 1.27)) hide)
-    )
-    (pin "1")
-    (pin "2")
-    (instances
-      (project "current_sink_dev"
-        (path "/695b42ec-77e0-4be3-bf4d-1fc5cfcb9ef1"
-          (reference "J2") (unit 1)
-        )
-      )
-    )
-  )
   (sheet (at 40.64 93.98) (size 57.15 29.21) (fields_autoplaced)
     (stroke (width 0.1524) (type solid))
@@
       (effects (font (size 1.27 1.27)) (justify left top))
     )
+    (instances
+      (project "current_sink_dev"
+        (path "/695b42ec-77e0-4be3-bf4d-1fc5cfcb9ef1" (page "6"))
+      )
+    )
+  )
+  (sheet (at 201.93 134.62) (size 58.42 29.21) (fields_autoplaced)
+    (stroke (width 0.1524) (type solid))
+    (fill (color 0 0 0 0.0000))
+    (property "Sheetname" "mechanical_components" (at 201.93 133.9084 0)
+      (effects (font (size 1.27 1.27)) (justify left bottom))
+    )
+    (property "Sheetfile" "mechanical_components.kicad_sch" (at 201.93 164.4146 0)
+      (effects (font (size 1.27 1.27)) (justify left top))
+    )
+    (instances
+      (project "current_sink_dev"
+        (path "/695b42ec-77e0-4be3-bf4d-1fc5cfcb9ef1" (page "7"))
+      )
+    )
+  )
+  (sheet (at 201.93 93.98) (size 58.42 29.21) (fields_autoplaced)
+    (stroke (width 0.1524) (type solid))
+    (fill (color 0 0 0 0.0000))
+    (property "Sheetname" "LCD_screen" (at 201.93 93.2684 0)
+      (effects (font (size 1.27 1.27)) (justify left bottom))
+    )
+    (property "Sheetfile" "LCD_screen.kicad_sch" (at 201.93 123.7746 0)
+      (effects (font (size 1.27 1.27)) (justify left top))
+    )

Commit message: Routing close to completion. Pending review.
Changed lines of the file:
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@@
 (kicad_sch (version 20230121) (generator eeschema)
   (paper "A3")
-  (sheet (at 40.64 93.98) (size 57.15 29.21) (fields_autoplaced)
+  (sheet (at 53.975 93.98) (size 57.15 29.21) (fields_autoplaced)
     (stroke (width 0.1524) (type solid))
     (fill (color 0 0 0 0.0000))
-    (property "Sheetname" "supply_gen" (at 40.64 93.2684 0)
+    (property "Sheetname" "supply_gen" (at 53.975 93.2684 0)
       (effects (font (size 1.27 1.27)) (justify left bottom))
     )
-    (property "Sheetfile" "supply_gen.kicad_sch" (at 40.64 123.7746 0)
+    (property "Sheetfile" "supply_gen.kicad_sch" (at 53.975 123.7746 0)
       (effects (font (size 1.27 1.27)) (justify left top))
     )
@@
     )
   )
-  (sheet (at 40.64 134.62) (size 57.15 29.21) (fields_autoplaced)
+  (sheet (at 53.975 134.62) (size 57.15 29.21) (fields_autoplaced)
     (stroke (width 0.1524) (type solid))
     (fill (color 0 0 0 0.0000))
-    (property "Sheetname" "uC_stage" (at 40.64 133.9084 0)
+    (property "Sheetname" "uC_stage" (at 53.975 133.9084 0)
       (effects (font (size 1.27 1.27)) (justify left bottom))
     )
-    (property "Sheetfile" "uC_stage.kicad_sch" (at 40.64 164.4146 0)
+    (property "Sheetfile" "uC_stage.kicad_sch" (at 53.975 164.4146 0)
       (effects (font (size 1.27 1.27)) (justify left top))
     )
