File: hardware/supply_gen.kicad_sch (KiCad schematic)
At the start: 5 parts, among them J2 USB_C_Receptacle_USB2.0, U5 PDSE1-S5-D5-M-TR

Commit message: Updates to structure of the schematic. Minor funcitonality adjustments.
Parts:
- added R1000: 0R, symbol Device:R_Small
- C7: renamed from C8; footprint (none) -> Capacitor_SMD:C_0805_2012Metric_Pad1.18x1.45mm_HandSolder
- C8: renamed from C7; footprint (none) -> Capacitor_SMD:C_0805_2012Metric_Pad1.18x1.45mm_HandSolder
- C9: footprint (none) -> Capacitor_SMD:C_0805_2012Metric_Pad1.18x1.45mm_HandSolder
- U5: footprint User_SupplyGen:PDSE1-S5-D5-M-TR -> User_SupplyGen:PDS1-M
Connections:
- net at C8.1, J2.A4 (VBUS), J2.A9 (VBUS)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: now also R1000.1
- net CC1 renamed USB_C_CC1_G
- net CC2 renamed USB_C_CC2_G
- net USB_C_D+ renamed USB_C_DPOS_G
- net USB_C_D- renamed USB_C_DNEG_G
- net supply_neg renamed -5V0_SUPPLY_G
- net supply_pos renamed 5V0_SUPPLY_G
- net 5V0_SUPPLY_G: now also R1000.2

Commit message: Began initial routing. Schematic still not fully complete.
Parts:
- R100: renamed from R1000; footprint (none) -> Resistor_SMD:R_0805_2012Metric_Pad1.20x1.40mm_HandSolder
- renumbered C7 to C100, C8 to C101, C9 to C102, U5 to U100
Other:
- note added: "In case U5 doesn't work as expected bridge the 5V"
Changed lines of the file:
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@@
     (stroke (width 0) (type default))
   )
+  (text "In case U5 doesn't work as expected bridge the 5V" (at 121.92 26.035 0)
+    (effects (font (size 1.27 1.27)) (justify left bottom))
+  )
   (global_label "5V0_SUPPLY_G" (shape bidirectional) (at 176.53 45.085 0) (fields_autoplaced)
     (effects (font (size 1.27 1.27)) (justify left))
@@
   (symbol (lib_id "power:GND1") (at 127 66.675 0) (unit 1)
     (in_bom yes) (on_board yes) (dnp no) (fields_autoplaced)
-    (property "Reference" "#PWR014" (at 127 73.025 0)
+    (property "Reference" "#PWR0101" (at 127 73.025 0)
       (effects (font (size 1.27 1.27)) hide)
     )
@@
       (project "current_sink_dev"
         (path "/695b42ec-77e0-4be3-bf4d-1fc5cfcb9ef1/02451f10-14c4-4640-81bd-2617f523efcf"
-          (reference "#PWR014") (unit 1)
+          (reference "#PWR0101") (unit 1)
         )
       )
@@
   (symbol (lib_id "power:GND") (at 201.295 57.15 0) (unit 1)
     (in_bom yes) (on_board yes) (dnp no) (fields_autoplaced)
-    (property "Reference" "#PWR013" (at 201.295 63.5 0)
+    (property "Reference" "#PWR0100" (at 201.295 63.5 0)
       (effects (font (size 1.27 1.27)) hide)
     )
@@
       (project "current_sink_dev"
         (path "/695b42ec-77e0-4be3-bf4d-1fc5cfcb9ef1/02451f10-14c4-4640-81bd-2617f523efcf"
-          (reference "#PWR013") (unit 1)
+          (reference "#PWR0100") (unit 1)
         )
       )
@@
   (symbol (lib_id "Device:C_Small") (at 127 53.975 0) (unit 1)
     (in_bom yes) (on_board yes) (dnp no) (fields_autoplaced)
-    (property "Reference" "C8" (at 129.54 53.3463 0)
+    (property "Reference" "C101" (at 129.54 53.3463 0)
       (effects (font (size 1.27 1.27)) (justify left))
     )
@@
       (project "current_sink_dev"
         (path "/695b42ec-77e0-4be3-bf4d-1fc5cfcb9ef1/02451f10-14c4-4640-81bd-2617f523efcf"
-          (reference "C8") (unit 1)
+          (reference "C101") (unit 1)
         )
       )
@@
       (project "current_sink_dev"
         (path "/695b42ec-77e0-4be3-bf4d-1fc5cfcb9ef1/02451f10-14c4-4640-81bd-2617f523efcf"
-          (reference "#PWR015") (unit 1)
+          (reference "#PWR0102") (unit 1)
         )
       )
@@
   (symbol (lib_id "Device:R_Small") (at 147.32 32.385 90) (unit 1)
     (in_bom yes) (on_board yes) (dnp no) (fields_autoplaced)
-    (property "Reference" "R1000" (at 147.32 27.94 90)
+    (property "Reference" "R100" (at 147.32 27.94 90)
       (effects (font (size 1.27 1.27)))
     )
@@
       (effects (font (size 1.27 1.27)))
     )
-    (property "Footprint" "" (at 147.32 32.385 0)
+    (property "Footprint" "Resistor_SMD:R_0805_2012Metric_Pad1.20x1.40mm_HandSolder" (at 147.32 32.385 0)
       (effects (font (size 1.27 1.27)) hide)
     )
@@
       (project "current_sink_dev"
         (path "/695b42ec-77e0-4be3-bf4d-1fc5cfcb9ef1/02451f10-14c4-4640-81bd-2617f523efcf"
-          (reference "R1000") (unit 1)
+          (reference "R100") (unit 1)
         )
       )
@@
       (project "current_sink_dev"
         (path "/695b42ec-77e0-4be3-bf4d-1fc5cfcb9ef1/02451f10-14c4-4640-81bd-2617f523efcf"
-          (reference "J1") (unit 1)
+          (reference "J100") (unit 1)
         )
       )
@@
   (symbol (lib_id "Device:C_Small") (at 165.735 48.895 0) (unit 1)
     (in_bom yes) (on_board yes) (dnp no) (fields_autoplaced)
-    (property "Reference" "C7" (at 168.275 48.2663 0)
+    (property "Reference" "C100" (at 168.275 48.2663 0)
       (effects (font (size 1.27 1.27)) (justify left))
     )
@@
       (project "current_sink_dev"
         (path "/695b42ec-77e0-4be3-bf4d-1fc5cfcb9ef1/02451f10-14c4-4640-81bd-2617f523efcf"
-          (reference "C7") (unit 1)
+          (reference "C100") (unit 1)
         )
       )
@@
   (symbol (lib_id "User_SupplyGen:PDSE1-S5-D5-M-TR") (at 140.335 46.355 0) (unit 1)
     (in_bom yes) (on_board yes) (dnp no) (fields_autoplaced)
-    (property "Reference" "U5" (at 147.0025 38.735 0)
+    (property "Reference" "U100" (at 147.0025 38.735 0)
       (effects (font (size 1.27 1.27)))
     )
@@
       (project "current_sink_dev"
         (path "/695b42ec-77e0-4be3-bf4d-1fc5cfcb9ef1/02451f10-14c4-4640-81bd-2617f523efcf"
-          (reference "U5") (unit 1)
+          (reference "U100") (unit 1)
         )
       )
@@
   (symbol (lib_id "Device:C_Small") (at 165.735 58.42 0) (unit 1)
     (in_bom yes) (on_board yes) (dnp no) (fields_autoplaced)
-    (property "Reference" "C9" (at 168.275 57.7913 0)
+    (property "Reference" "C102" (at 168.275 57.7913 0)
       (effects (font (size 1.27 1.27)) (justify left))
     )
@@
       (project "current_sink_dev"
         (path "/695b42ec-77e0-4be3-bf4d-1fc5cfcb9ef1/02451f10-14c4-4640-81bd-2617f523efcf"
-          (reference "C9") (unit 1)
-        )
-      )
+          (reference "C102") (unit 1)
+        )
+      )

Commit message: Routing close to completion. Pending review.
Parts:
- added J503: 5V_IN, Connector_PinSocket_2.54mm:PinSocket_1x02_P2.54mm_Vertical, symbol Connector:Conn_01x02_Socket
- added TP500, TP501, TP502: ~, TestPoint:TestPoint_Pad_D1.0mm, symbol Connector:TestPoint
Connections:
- net GND1 is gone; now on net GND: C101.2, U100.1 (GND)
- net -5V0_SUPPLY_G: now also TP501.1
- net 5V0_SUPPLY_G: now also TP500.1
- net GND: now also J503.2 (Pin_2)
- net usb5v_l: now reaches C101.1, J2.A4 (VBUS), J2.A9 (VBUS), J2.B4 (VBUS), J2.B9 (VBUS), R100.1, U100.2 (VIN)
- net usb5v_l: now also J503.1 (Pin_1), TP502.1
Other:
- moved on the sheet: J2
